File: 2019_Dashboard_2_4_19.brd (EAGLE design)
At the start: 93.7 x 49.2 mm, 60 parts, among them IC1 MCP23017SO, Q1 TN0602N3, Q2 TN0602N3, Q3 TN0602N3, Q4 TN0602N3, Q5 TN0602N3, U1 TLC59281, Y1 16MHz

Commit message: Add files via upload
Dear lord Jesus please let it be done
Parts:
- moved D14 109.7 mm to (128.3, 48.3)
- moved Q1 63.7 mm to (69.8, 69.8)
- moved Q5 15.7 mm to (124.5, 34.3)
- moved Q4 12.0 mm to (96.5, 68.6)
- moved U1 5.68 mm to (78.7, 69.8)
- moved Q2 4.58 mm to (105.4, 68.6)
- moved D1 3.81 mm to (54.6, 77.5)
- moved D10 3.81 mm to (111.8, 77.5)
- moved D11 3.81 mm to (118.1, 77.5)
- moved D12 3.81 mm to (124.5, 77.5)
- moved D2 3.81 mm to (61.0, 77.5)
- moved D3 3.81 mm to (67.3, 77.5)
- moved D4 3.81 mm to (73.7, 77.5)
- moved D5 3.81 mm to (80.0, 77.5)
- moved D6 3.81 mm to (86.4, 77.5)
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Routing:
- net VCC: track 263.1 -> 151.5 mm, vias 4 -> 5
- net N$11: track 60.6 -> 11.7 mm
- net RESET: track 47.8 -> 81.3 mm, vias 3 -> 1
- net N$28: track 51.9 -> 26.3 mm, vias 0 -> 2
- net N$6: track 76.2 -> 52.0 mm, vias 1 -> 0
- net N$50: track 48.6 -> 28.0 mm
- net GND: track 229.7 -> 212.9 mm, vias 12 -> 33
- net LAUNCH: track 47.1 -> 62.6 mm, vias 2 -> 1
- net CANL: track 31.1 -> 45.8 mm
- net N$31: track 28.8 -> 42.1 mm
- net HEAT: track 46.2 -> 33.6 mm, vias 3 -> 0
- net N$13: track 25.8 -> 38.5 mm, vias 0 -> 1
- net N$47: track 31.0 -> 43.4 mm
- net N$5: track 65.7 -> 77.4 mm
- net N$8: track 48.9 -> 59.0 mm, vias 2 -> 1
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Other:
- board size 93.7 x 49.2 mm -> 93.7 x 53 mm
